File: pcb/commissioner/commissioner.kicad_sch (KiCad schematic)
At the start: 0 parts

Commit message: arduino case, kicad basic setup
Parts:
- added U1: ESP32-S3-WROOM-1, RF_Module:ESP32-S3-WROOM-1U, symbol RF_Module:ESP32-S3-WROOM-1
- added U2: XBee3_SMT, XBee3:XBee3_SMT, symbol XBee3:XBee3_SMT
Connections:
- new net: U1.1 (GND), U1.40 (GND), U1.41 (GND)
- new net GND: U2.1 (GND), U2.10 (GND), U2.12 (GND), U2.21 (GND), U2.32 (GND), U2.34 (GND)
