File: hardware/pcb/coordinator/coordinator.kicad_sch (KiCad schematic)
At the start: 11 parts, among them J1 XBee3 TH, J2 XBee3 TH, J3 WIZ820IO TH, J4 WIZ820IO TH, J5 USB-C Power Breakout, SW1 SW_Push, U1 ESP32-C3_SUPERMINI_TH

Commit message: All PCBs finalized, ready to order
Parts:
- removed D1: LED, LED_THT:LED_D5.0mm, symbol Device:LED
- removed J5: USB-C Power Breakout, Connector_PinHeader_2.54mm:PinHeader_1x04_P2.54mm_Vertical, symbol Connector:Conn_01x04_Pin
- removed SW1: SW_Push, Button_Switch_THT:SW_PUSH_6mm, symbol Switch:SW_Push
- added J6: USB-C, Connector_PinSocket_2.54mm:PinSocket_1x08_P2.54mm_Vertical, symbol Connector:Conn_01x08_Socket
- J1, J2: footprint Connector_PinHeader_2.00mm:PinHeader_1x10_P2.00mm_Vertical -> Connector_PinSocket_2.00mm:PinSocket_1x10_P2.00mm_Vertical
- J3, J4: footprint Connector_PinHeader_2.54mm:PinHeader_1x06_P2.54mm_Vertical -> Connector_PinSocket_2.54mm:PinSocket_1x06_P2.54mm_Vertical
Connections:
- net GND: now also J6.1 (Pin_1)
- net at R4.1: now also J6.8 (Pin_8)
- net at U1.5V: now also J6.2 (Pin_2)
- net at R2.1: now also J6.4 (Pin_4)
- no-connect marks 19 -> 25
Other:
- moved on the sheet: R2, R4
