File: hardware/pcb/coordinator/coordinator.kicad_pcb (KiCad board)
At the start: 2 copper layers, 53 x 73.2 mm, 15 parts, among them J1 XBee3 TH, J2 XBee3 TH, J3 WIZ820IO TH, J4 WIZ820IO TH, J5 USB-C Power Breakout, SW1 SW_Push, U1 ESP32-C3_SUPERMINI_TH

Commit message: Joiner PCB began
Parts:
- R1, R2, R4: footprint Resistor_THT:R_Axial_DIN0207_L6.3mm_D2.5mm_P2.54mm_Vertical -> Resistor_THT:R_Axial_DIN0207_L6.3mm_D2.5mm_P7.62mm_Horizontal
- moved R4 5.98 mm to (104.2, 115.5), turned to 90 degrees
- moved R1 5.21 mm to (99.0, 64.2), turned to -90 degrees
- moved R2 2.87 mm to (98.0, 115.6), turned to 90 degrees
- moved J5 2.68 mm to (109.6, 114.8)
Routing:
- net Net-(J5-CC2): track 16.3 -> 9.12 mm, vias 1 -> 0
- net Net-(J5-CC1): track 9.47 -> 15.1 mm, vias 1 -> 0
- net Net-(J5-VBUS): track 38.7 -> 34.1 mm
- net +3.3V: track 104.4 -> 100.7 mm
- net Net-(J1-RST): track 6.65 -> 7.43 mm

Commit message: Made Joiner PCB Progress
Other:
- board text added: "M2"
Changed lines of the file:
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@@
 		(layer "Edge.Cuts")
+	)
+	(gr_text "M2"
+		(at 92 63.2 0)
+		(layer "F.Cu")
+		(effects
+			(font
+				(size 1.5 1.5)
+				(thickness 0.3)
+				(bold yes)
+			)
+			(justify left bottom)
+		)
+	)
+	(gr_text "M2"
+		(at 92 120.8 0)
+		(layer "F.Cu")
+		(effects
+			(font
+				(size 1.5 1.5)
+				(thickness 0.3)
+				(bold yes)
+			)
+			(justify left bottom)
+		)
+	)
+	(gr_text "M2"
+		(at 137 63.2 0)
+		(layer "F.Cu")
+		(effects
+			(font
+				(size 1.5 1.5)
+				(thickness 0.3)
+				(bold yes)
+			)
+			(justify left bottom)
+		)
+	)
+	(gr_text "M2"
+		(at 137.6 121 0)
+		(layer "F.Cu")
+		(effects
+			(font
+				(size 1.5 1.5)
+				(thickness 0.3)
+				(bold yes)
+			)
+			(justify left bottom)
+		)
 	)
 	(segment
