File: hardware/pcb/coordinator/coordinator.kicad_pcb (KiCad board)
At the start: 2 copper layers, 53 x 73.2 mm, 15 parts, among them J1 XBee3 TH, J2 XBee3 TH, J3 WIZ820IO TH, J4 WIZ820IO TH, J5 USB-C Power Breakout, SW1 SW_Push, U1 ESP32-C3_SUPERMINI_TH

Commit message: All PCBs finalized, ready to order
Parts:
- removed D1: LED, LED_THT:LED_D5.0mm
- removed J5: USB-C Power Breakout, Connector_PinHeader_2.54mm:PinHeader_1x04_P2.54mm_Vertical
- removed the REF** at (93.8, 58.4)
- removed the REF** at (139.2, 124.0)
- removed the REF** at (93.8, 124.0)
- removed the REF** at (139.0, 58.4)
- removed SW1: SW_Push, Button_Switch_THT:SW_PUSH_6mm
- added J6: USB-C, Connector_PinSocket_2.54mm:PinSocket_1x08_P2.54mm_Vertical, F.Cu at (97.8, 84.3)
- added REF**: M2, MountingHole:MountingHole_2.2mm_M2, F.Cu at (93.2, 124.0)
- added REF**: M2, MountingHole:MountingHole_2.2mm_M2, F.Cu at (93.2, 59.2)
- added REF**: M2, MountingHole:MountingHole_2.2mm_M2, F.Cu at (139.8, 123.8)
- added REF**: M2, MountingHole:MountingHole_2.2mm_M2, F.Cu at (139.8, 59.0)
- J1, J2: footprint Connector_PinHeader_2.00mm:PinHeader_1x10_P2.00mm_Vertical -> Connector_PinSocket_2.00mm:PinSocket_1x10_P2.00mm_Vertical
- J3, J4: footprint Connector_PinHeader_2.54mm:PinHeader_1x06_P2.54mm_Vertical -> Connector_PinSocket_2.54mm:PinSocket_1x06_P2.54mm_Vertical
- moved R1 51.8 mm to (112.4, 114.2)
- moved R2 6.52 mm to (99.8, 121.9)
- moved R4 6.52 mm to (106.0, 121.8)
Connections:
- U1 pad 3: Net-(U1-GPIO3) -> unconnected-(U1-GPIO3-Pad3)
- U1 pad 4: Net-(D1-A) -> unconnected-(U1-GPIO4-Pad4)
Routing:
- net Net-(J1-RST): track 7.43 -> 57.6 mm, vias 0 -> 2
- net Net-(U1-GPIO3): track 39.4 -> 0.00 mm
- net Net-(D1-A): track 29.7 -> 0.00 mm
- net Net-(J6-Pin_8): track 9.12 -> 28.7 mm
- net Net-(J6-Pin_4): track 15.1 -> 31.7 mm
- net Net-(J6-Pin_2): track 34.1 -> 42.0 mm, vias 0 -> 3
- net GND: track 12.8 -> 14.8 mm
- net +3.3V: track 100.7 -> 102.4 mm, vias 6 -> 4
Other:
- board size 53 x 73.2 mm -> 53 x 74 mm
- board text added: "53mm x 74mm"
- board text removed: "M2"
